File: flash.kicad_pcb (KiCad board)
At the start: 4 copper layers, 62.5 x 49 mm, 75 parts, among them J1 USB_C_Receptacle_USB2.0_14P, J2 Power, J3 AOUT, J4 BOUT, J5 LSIN, J6 LSOUT, SW1 SW_DIP_x04, SW2 CAS-D20TA, SW3 SW_Nidec_CAS-120A1, SW4 SW_DIP_x03, SW5 SW_DIP_x03, SW6 Reset Button, U1 LDK130M18R, U2 LDK130M25R, U3 AP2112K-3.3, U4 USBLC6-2SC6, U5 FT2232HL, U6 SN74LVC8T245PWR, U7 SN74LVC8T245PWR, U8 93LCxxBxxOT, Y1 SCTF SX3M12.000M20F30TNN

Commit message: MondayAkiba
Parts:
- added C15: 10pF, Capacitor_SMD:C_0603_1608Metric_Pad1.08x0.95mm_HandSolder, F.Cu at (147.8, 100.8)
- C14: value 0.01uF -> 10pF
- Y1: value SCTF SX3M12.000M20F30TNN -> Crystal_GND24
- moved J2 25.9 mm to (183.5, 125.7), turned to -90 degrees
- moved SW3 19.8 mm to (187.5, 97.5), turned to 180 degrees
- moved C14 6.32 mm to (151.0, 105.5), turned to -90 degrees
- moved R10 1.75 mm to (159.0, 125.0)
- moved Y1 1.60 mm to (147.8, 104.5), turned to 90 degrees
- moved C10 1.28 mm to (179.1, 102.2)
- moved C11 1.28 mm to (183.1, 102.2)
- moved C12 1.28 mm to (179.1, 112.2)
- moved C13 1.28 mm to (183.1, 112.2)
- moved U6 1.28 mm to (181.1, 107.2)
- moved U7 1.28 mm to (181.1, 117.2)
- moved C32 1.25 mm to (167.5, 125.0)
- moved SW4 1.25 mm to (163.0, 125.0)
- moved C20 1.18 mm to (169.0, 115.1), turned to 180 degrees
- moved J5 0.50 mm to (172.7, 103.6)
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- renumbered C9 to C10, C10 to C11, C11 to C12, C12 to C13, C15 to C16, C16 to C17, C17 to C21, C21 to C22, C22 to C23, C23 to C24, C32 to C25, C24 to C26, C25 to C27, C26 to C28, C27 to C29, C28 to C30, C29 to C31, C31 to C32, C30 to C33, C13 to C9, R14 to R10, R10 to R11, R11 to R12, R12 to R13, R13 to R14, SW6 to SW4, SW4 to SW5, SW5 to SW6
Connections:
- C14 pad 2: 3.3V -> XCSO
- U5 pad 3: unconnected-(U5-OSCO-Pad3) -> XCSO
- Y1 pad 1: 3.3V -> XCSO
- Y1 pad 4: 3.3V -> GND
Routing:
- net 3.3V: track 136.5 -> 205.6 mm, vias 14 -> 16
- net BD1: track 7.35 -> 40.9 mm, vias 0 -> 2
- net DIR1: track 0.00 -> 33.1 mm
- net GND: track 76.3 -> 106.6 mm, vias 206 -> 321
- net PWREN: track 1.53 -> 30.8 mm
- net AC7: track 0.00 -> 24.1 mm, vias 0 -> 1
- net SUSPEND: track 0.00 -> 23.0 mm, vias 0 -> 1
- net BD0: track 10.1 -> 32.1 mm, vias 0 -> 2
- net ISOLATE: track 0.00 -> 21.6 mm, vias 0 -> 2
- net AC6: track 0.00 -> 21.0 mm, vias 0 -> 1
- net AC5: track 0.00 -> 18.7 mm, vias 0 -> 1
- net AC4: track 0.00 -> 18.3 mm, vias 0 -> 1
- net AC3: track 0.00 -> 17.5 mm, vias 0 -> 1
- net DIR2: track 0.00 -> 17.2 mm
- net AC2: track 0.00 -> 16.8 mm, vias 0 -> 1
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Other:
- board text added: "<-- ISOLATE"
- board text added: "<-LS2-> <-LS1->"
- board text added: "BD1->BD2 BD1->4.7k BD0->4.7k"
- board text added: "LS1 r 1 2r 3 4r 5 6r 7 8 LS2"
- board text added: "PWREN VVAR 3V3"
- board text added: "RESET"
- board text added: "SUSP GND GND"
