File: flash.kicad_sch (KiCad schematic)
At the start: 71 parts, among them J1 USB_C_Receptacle_USB2.0_14P, J2 Power, J3 AOUT, J4 BOUT, J5 LSIN, J6 LSOUT, SW1 SW_DIP_x04, SW2 CAS-D20TA, SW3 SW_Nidec_CAS-120A1, SW4 SW_DIP_x03, SW5 SW_DIP_x03, SW6 Reset Button, U1 LDK130M18R, U2 LDK130M25R, U3 AP2112K-3.3, U4 USBLC6-2SC6, U5 FT2232HL, U6 SN74LVC8T245PWR, U7 SN74LVC8T245PWR, U8 93LCxxBxxOT, Y1 SCTF SX3M12.000M20F30TNN

Commit message: MondayAkiba
Parts:
- removed Y1: SCTF SX3M12.000M20F30TNN, Crystal:Crystal_SMD_3225-4Pin_3.2x2.5mm_HandSoldering, symbol Oscillator:XO32
- added C15: 10pF, Capacitor_SMD:C_0603_1608Metric_Pad1.08x0.95mm_HandSolder, symbol Device:C_Small
- added Y1: Crystal_GND24, Crystal:Crystal_SMD_3225-4Pin_3.2x2.5mm_HandSoldering, symbol Device:Crystal_GND24
- C14: value 0.01uF -> 10pF
- renumbered C9 to C10, C10 to C11, C11 to C12, C12 to C13, C15 to C16, C16 to C17, C17 to C21, C21 to C22, C22 to C23, C23 to C24, C32 to C25, C24 to C26, C25 to C27, C26 to C28, C27 to C29, C28 to C30, C29 to C31, C31 to C32, C30 to C33, C13 to C9, R14 to R10, R10 to R11, R11 to R12, R12 to R13, R13 to R14, SW6 to SW4, SW4 to SW5, SW5 to SW6
Connections:
- net 3.3V: no longer C14.2
- net GND: now also C15.2, Y1.2 (G), Y1.4 (G)
- net XCSI: now also C15.1, Y1.3
- net XCSO: now reaches U5.3 (OSCO)
- net XCSO: now also C14.2, Y1.1
- no-connect marks 5 -> 4
Other:
- moved on the sheet: C16, R6, R7, R8, R9, U8
